File: head-interface.kicad_pcb (KiCad board)
At the start: 2 copper layers, 51.1 x 19.6 mm, 10 parts, among them J1 NOZ, J2 FANS, J3 MOTOR_IN, J4 THERM, J5 HEATER, J6 PART_FAN, J7 FAN, J8 MOTOR

Commit message: rc1
Connections:
- H1 pad 1: (no net) -> GND
- H2 pad 1: (no net) -> GND
Routing:
- net GND: vias 0 -> 21
- added copper zone on B.Cu, net GND
- added copper zone on F.Cu, net GND
Changed lines of the file:
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@@
   (net 11 "Net-(J2-Pad1)")
   (net 12 "Net-(J2-Pad2)")
+  (net 13 "GND")
   (footprint "Connector_JST:JST_EH_B4B-EH-A_1x04_P2.50mm_Vertical" (layer "F.Cu")
     (at 90.825 57.15 180)
@@
     (fp_circle (center 0 0) (end 3.2 0) (layer "Cmts.User") (width 0.15) (fill none))
     (fp_circle (center 0 0) (end 3.45 0) (layer "F.CrtYd") (width 0.05) (fill none))
-    (pad "1" thru_hole circle locked (at 0 0) (size 6.4 6.4) (drill 3.2) (layers *.Cu *.Mask))
+    (pad "1" thru_hole circle locked (at 0 0) (size 6 6) (drill 3.2) (layers *.Cu *.Mask)
+      (net 13 "GND") (pinfunction "1") (pintype "input") (zone_connect 2))
   )
   (footprint "Connector_JST:JST_PH_B2B-PH-K_1x02_P2.00mm_Vertical" (layer "F.Cu")
@@
     (fp_circle (center 0 0) (end 3.2 0) (layer "Cmts.User") (width 0.15) (fill none))
     (fp_circle (center 0 0) (end 3.45 0) (layer "F.CrtYd") (width 0.05) (fill none))
-    (pad "1" thru_hole circle locked (at 0 0) (size 6.4 6.4) (drill 3.2) (layers *.Cu *.Mask))
+    (pad "1" thru_hole circle locked (at 0 0) (size 6 6) (drill 3.2) (layers *.Cu *.Mask)
+      (net 13 "GND") (pinfunction "1") (pintype "input") (zone_connect 2))
   )
   (footprint "Connector_JST:JST_EH_B4B-EH-A_1x04_P2.50mm_Vertical" (layer "F.Cu")
@@
     (effects (font (size 1 1) (thickness 0.15)) (justify mirror))
   )
-  (segment (start 78.6 42.4) (end 78.6 51.6) (width 0.5) (layer "F.Cu") (net 1))
-  (segment (start 78.6 51.6) (end 79.2 52.2) (width 0.5) (layer "F.Cu") (net 1))
-  (segment (start 76.6 52.1) (end 76.7 52.2) (width 0.5) (layer "F.Cu") (net 2))
-  (segment (start 76.6 42.4) (end 76.6 52.1) (width 0.5) (layer "F.Cu") (net 2))
-  (segment (start 69.3 54.9) (end 60.6 46.2) (width 0.5) (layer "F.Cu") (net 3))
-  (segment (start 60.6 46.2) (end 60.6 42.4) (width 0.5) (layer "F.Cu") (net 3))
-  (segment (start 69.3 57.15) (end 69.3 54.9) (width 0.5) (layer "F.Cu") (net 3))
-  (segment (start 62.6 46.6) (end 62.6 42.4) (width 0.5) (layer "F.Cu") (net 4))
-  (segment (start 71.8 57.15) (end 71.8 55.8) (width 0.5) (layer "F.Cu") (net 4))
-  (segment (start 71.8 55.8) (end 62.6 46.6) (width 0.5) (layer "F.Cu") (net 4))
-  (segment (start 71.3 50.3) (end 71.3 45.2) (width 1) (layer "F.Cu") (net 5))
-  (segment (start 76.8 55.8) (end 71.3 50.3) (width 1) (layer "F.Cu") (net 5))
-  (segment (start 76.8 57.15) (end 76.8 55.8) (width 1) (layer "F.Cu") (net 5))
-  (segment (start 74.3 55.7) (end 67.8 49.2) (width 1) (layer "F.Cu") (net 6))
-  (segment (start 74.3 57.15) (end 74.3 55.7) (width 1) (layer "F.Cu") (net 6))
-  (segment (start 67.8 49.2) (end 67.8 45.2) (width 1) (layer "F.Cu") (net 6))
-  (segment (start 90.825 54.775) (end 99.15 46.45) (width 1) (layer "F.Cu") (net 7))
-  (segment (start 99.15 46.45) (end 99.15 42.95) (width 1) (layer "F.Cu") (net 7))
-  (segment (start 90.825 57.15) (end 90.825 54.775) (width 1) (layer "F.Cu") (net 7))
-  (segment (start 99.15 42.95) (end 99.1 42.9) (width 1) (layer "F.Cu") (net 7))
-  (segment (start 88.325 55.275) (end 96.65 46.95) (width 1) (layer "F.Cu") (net 8))
-  (segment (start 88.325 57.15) (end 88.325 55.275) (width 1) (layer "F.Cu") (net 8))
-  (segment (start 96.65 42.95) (end 96.6 42.9) (width 1) (layer "F.Cu") (net 8))
-  (segment (start 96.65 46.95) (end 96.65 42.95) (width 1) (layer "F.Cu") (net 8))
-  (segment (start 94.15 42.95) (end 94.1 42.9) (width 1) (layer "F.Cu") (net 9))
-  (segment (start 94.15 47.45) (end 94.15 42.95) (width 1) (layer "F.Cu") (net 9))
-  (segment (start 85.825 55.775) (end 94.15 47.45) (width 1) (layer "F.Cu") (net 9))
-  (segment (start 85.825 57.15) (end 85.825 55.775) (width 1) (layer "F.Cu") (net 9))
-  (segment (start 91.65 47.95) (end 91.65 42.95) (width 1) (layer "F.Cu") (net 10))
-  (segment (start 83.325 56.275) (end 91.65 47.95) (width 1) (layer "F.Cu") (net 10))
-  (segment (start 83.325 57.15) (end 83.325 56.275) (width 1) (layer "F.Cu") (net 10))
-  (segment (start 91.65 42.95) (end 91.6 42.9) (width 1) (layer "F.Cu") (net 10))
-  (segment (start 85.8 50.6) (end 85.8 42.4) (width 0.5) (layer "F.Cu") (net 11))
-  (segment (start 84.2 52.2) (end 85.8 50.6) (width 0.5) (layer "F.Cu") (net 11))
-  (segment (start 81.8 52.2) (end 83.8 50.2) (width 0.5) (layer "F.Cu") (net 12))
-  (segment (start 81.7 52.2) (end 81.8 52.2) (width 0.5) (layer "F.Cu") (net 12))
-  (segment (start 83.8 50.2) (end 83.8 42.4) (width 0.5) (layer "F.Cu") (net 12))
+  (segment (start 78.6 42.4) (end 78.6 51.6) (width 0.5) (layer "B.Cu") (net 1))
+  (segment (start 78.6 51.6) (end 79.2 52.2) (width 0.5) (layer "B.Cu") (net 1))
+  (segment (start 76.6 52.1) (end 76.7 52.2) (width 0.5) (layer "B.Cu") (net 2))
+  (segment (start 76.6 42.4) (end 76.6 52.1) (width 0.5) (layer "B.Cu") (net 2))
+  (segment (start 69.3 54.9) (end 60.6 46.2) (width 0.5) (layer "B.Cu") (net 3))
+  (segment (start 60.6 46.2) (end 60.6 42.4) (width 0.5) (layer "B.Cu") (net 3))
+  (segment (start 69.3 57.15) (end 69.3 54.9) (width 0.5) (layer "B.Cu") (net 3))
+  (segment (start 62.6 46.6) (end 62.6 42.4) (width 0.5) (layer "B.Cu") (net 4))
+  (segment (start 71.8 57.15) (end 71.8 55.8) (width 0.5) (layer "B.Cu") (net 4))
+  (segment (start 71.8 55.8) (end 62.6 46.6) (width 0.5) (layer "B.Cu") (net 4))
+  (segment (start 71.3 50.3) (end 71.3 45.2) (width 1) (layer "B.Cu") (net 5))
+  (segment (start 76.8 55.8) (end 71.3 50.3) (width 1) (layer "B.Cu") (net 5))
+  (segment (start 76.8 57.15) (end 76.8 55.8) (width 1) (layer "B.Cu") (net 5))
+  (segment (start 74.3 55.7) (end 67.8 49.2) (width 1) (layer "B.Cu") (net 6))
+  (segment (start 74.3 57.15) (end 74.3 55.7) (width 1) (layer "B.Cu") (net 6))
+  (segment (start 67.8 49.2) (end 67.8 45.2) (width 1) (layer "B.Cu") (net 6))
+  (segment (start 90.825 54.775) (end 99.15 46.45) (width 1) (layer "B.Cu") (net 7))
+  (segment (start 99.15 46.45) (end 99.15 42.95) (width 1) (layer "B.Cu") (net 7))
+  (segment (start 90.825 57.15) (end 90.825 54.775) (width 1) (layer "B.Cu") (net 7))
+  (segment (start 99.15 42.95) (end 99.1 42.9) (width 1) (layer "B.Cu") (net 7))
+  (segment (start 88.325 55.275) (end 96.65 46.95) (width 1) (layer "B.Cu") (net 8))
+  (segment (start 88.325 57.15) (end 88.325 55.275) (width 1) (layer "B.Cu") (net 8))
+  (segment (start 96.65 42.95) (end 96.6 42.9) (width 1) (layer "B.Cu") (net 8))
+  (segment (start 96.65 46.95) (end 96.65 42.95) (width 1) (layer "B.Cu") (net 8))
+  (segment (start 94.15 42.95) (end 94.1 42.9) (width 1) (layer "B.Cu") (net 9))
+  (segment (start 94.15 47.45) (end 94.15 42.95) (width 1) (layer "B.Cu") (net 9))
+  (segment (start 85.825 55.775) (end 94.15 47.45) (width 1) (layer "B.Cu") (net 9))
+  (segment (start 85.825 57.15) (end 85.825 55.775) (width 1) (layer "B.Cu") (net 9))
+  (segment (start 91.65 47.95) (end 91.65 42.95) (width 1) (layer "B.Cu") (net 10))
+  (segment (start 83.325 56.275) (end 91.65 47.95) (width 1) (layer "B.Cu") (net 10))
+  (segment (start 83.325 57.15) (end 83.325 56.275) (width 1) (layer "B.Cu") (net 10))
+  (segment (start 91.65 42.95) (end 91.6 42.9) (width 1) (layer "B.Cu") (net 10))
+  (segment (start 85.8 50.6) (end 85.8 42.4) (width 0.5) (layer "B.Cu") (net 11))
+  (segment (start 84.2 52.2) (end 85.8 50.6) (width 0.5) (layer "B.Cu") (net 11))
+  (segment (start 81.8 52.2) (end 83.8 50.2) (width 0.5) (layer "B.Cu") (net 12))
+  (segment (start 81.7 52.2) (end 81.8 52.2) (width 0.5) (layer "B.Cu") (net 12))
+  (segment (start 83.8 50.2) (end 83.8 42.4) (width 0.5) (layer "B.Cu") (net 12))
+  (via (at 82.65 54.35) (size 0.8) (drill 0.4) (layers "F.Cu" "B.Cu") (free) (net 13))
+  (via (at 101.25 41.325) (size 0.8) (drill 0.4) (layers "F.Cu" "B.Cu") (free) (net 13))
+  (via (at 72.875 49.675) (size 0.8) (drill 0.4) (layers "F.Cu" "B.Cu") (free) (net 13))
+  (via (at 65.825 58.45) (size 0.8) (drill 0.4) (layers "F.Cu" "B.Cu") (free) (net 13))
+  (via (at 92.9 55.5) (size 0.8) (drill 0.4) (layers "F.Cu" "B.Cu") (free) (net 13))
+  (via (at 94.125 58.45) (size 0.8) (drill 0.4) (layers "F.Cu" "B.Cu") (free) (net 13))
+  (via (at 65.45 41.325) (size 0.8) (drill 0.4) (layers "F.Cu" "B.Cu") (free) (net 13))
+  (via (at 89.775 47.1) (size 0.8) (drill 0.4) (layers "F.Cu" "B.Cu") (free) (net 13))
+  (via (at 64.6 46.325) (size 0.8) (drill 0.4) (layers "F.Cu" "B.Cu") (free) (net 13))
+  (via (at 63.65 51.1) (size 0.8) (drill 0.4) (layers "F.Cu" "B.Cu") (free) (net 13))
+  (via (at 77.475 54.375) (size 0.8) (drill 0.4) (layers "F.Cu" "B.Cu") (free) (net 13))
+  (via (at 66.35 47.85) (size 0.8) (drill 0.4) (layers "F.Cu" "B.Cu") (free) (net 13))
+  (via (at 88.425 41.325) (size 0.8) (drill 0.4) (layers "F.Cu" "B.Cu") (free) (net 13))
+  (via (at 79.95 49.4) (size 0.8) (drill 0.4) (layers "F.Cu" "B.Cu") (free) (net 13))
+  (via (at 87.55 49.325) (size 0.8) (drill 0.4) (layers "F.Cu" "B.Cu") (free) (net 13))
+  (via (at 82.45 49.4) (size 0.8) (drill 0.4) (layers "F.Cu" "B.Cu") (free) (net 13))
+  (via (at 67.225 55.5) (size 0.8) (drill 0.4) (layers "F.Cu" "B.Cu") (free) (net 13))
+  (via (at 79.975 58.45) (size 0.8) (drill 0.4) (layers "F.Cu" "B.Cu") (free) (net 13))
+  (via (at 59.05 41.325) (size 0.8) (drill 0.4) (layers "F.Cu" "B.Cu") (free) (net 13))
+  (via (at 73.8 41.325) (size 0.8) (drill 0.4) (layers "F.Cu" "B.Cu") (free) (net 13))
+  (via (at 74.625 50.675) (size 0.8) (drill 0.4) (layers "F.Cu" "B.Cu") (free) (net 13))
+  (zone (net 13) (net_name "GND") (layers F&B.Cu) (hatch edge 0.508)
+    (connect_pads (clearance 0.508))
+    (min_thickness 0.254) (filled_areas_thickness no)
+    (fill yes (thermal_gap 0.508) (thermal_bridge_width 0.508))
+    (polygon
+      (pts
+        (xy 108.975 63.55)
+        (xy 51.575 63.55)
+        (xy 51.575 37.35)
+        (xy 108.9 37.35)
+      )
+    )
+  )
 )
