File: head-interface.kicad_pcb (KiCad board)
At the start: 2 copper layers, 51.1 x 19.6 mm, 10 parts, among them J1 NOZ, J2 FANS, J3 MOTOR_IN, J4 THERM, J5 HEATER, J6 PART_FAN, J7 FAN, J8 MOTOR

Commit message: tweaks
Parts:
- moved H1 39.4 mm to (78.0, 84.9)
- moved H2 39.4 mm to (122.0, 84.9)
- moved J1 39.4 mm to (96.8, 91.0)
- moved J3 39.4 mm to (110.8, 91.0)
- moved J4 39.4 mm to (80.6, 76.3)
- moved J6 39.4 mm to (103.8, 76.3)
- moved J7 39.4 mm to (96.6, 76.3)
- moved J8 39.4 mm to (119.1, 76.8)
- moved J2 39.4 mm to (104.2, 86.1)
- moved J5 39.4 mm to (91.3, 79.1)
Other:
- board text added: "(0,-20) X-CENTER FLIP DOWEL"
- board text added: "(0,0) X-CENTER FLIP DOWEL"
